File: fiat_light_relay/fiat_light_relay.kicad_pcb (KiCad board)
At the start: 2 copper layers, 52 x 52 mm, 11 parts, among them J4 Conn_01x06, J5 Conn_01x01

Commit message: Added some new projects
Parts:
- moved J4 0.25 mm to (10.0, 33.0)
- moved J5 0.25 mm to (42.0, 33.0)
