File: scrubotron/main_board/tape_jar.kicad_sch (KiCad schematic)
At the start: 28 parts, among them J1 Battery, J2 AudioJack3, J4 AudioJack3, SW1 SW_SPDT, U1 TL072, U2 NE5532

Commit message: Updated schematic
Parts:
- J2: value AudioJack3 -> Audio Output
- J4: value AudioJack3 -> Wand Input
- SW1: value SW_SPDT -> Power Switch
Other:
- note added: "55x Gain"
- note added: "C10 provides bulk capacitance in case the battery can't keep up with current spikes"
- note added: "C3 prevents high frequency oscillation by removing phase shift in the feedback network"
- note added: "Capacitors remove the DC component from the signal"
- note added: "Create virtual ground at 4.5V with voltage divider"
- note added: "Headphone Amplifier (no gain)"
- note added: "NAB Equalization (100-1000x gain according to freq)"
- note added: "Resistors try to prevent damage to the op amp from high currents such as from ESD"
- note added: "Volume Control"
- title: (none) -> Scrubotron
- moved on the sheet: C1, C10, C2, C3, C4, C5, C6, C8, J1, J2, J4, R1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
